File: projects/max_bell/max_bell_eagle/max_bell.sch (EAGLE design)
At the start: 19 parts

Commit message: updates to max_bell
Parts:
- removed GPIO: (no value), pinhead:PINHD-1X8/90
- added JP1: (no value), pinhead:PINHD-1X10
- added R5: 10K, rcl:R-US_0309/12
- added U$5: SWITCH_MOMENTARY, fritz:SWITCH_MOMENTARY
- R2: value 1K -> 10K
Connections:
- net GND: now also JP1.1, U$5.2; no longer U$4.2
- net GPIO_0: now also JP1.3; no longer GPIO.1
- net GPIO_1: now also JP1.4; no longer GPIO.2
- net GPIO_2: now also JP1.5, R5.1, U$5.1; no longer GPIO.3
- net GPIO_3: now also JP1.6; no longer GPIO.4
- net GPIO_4: now also JP1.7; no longer GPIO.5
- net GPIO_5: now also JP1.8; no longer GPIO.6
- net GPIO_6: now also JP1.9; no longer GPIO.7
- net GPIO_7: now also JP1.10; no longer GPIO.8
- net ICSPCLK: now also U$1.RA1/ICSPCLK
- net ICSPDAT: now also U$1.RA0/ICSPDAT
- net VDD: now also JP1.2, R5.2, U$4.2
Changed lines of the file:
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@@
 <part name="U$1" library="fritz" deviceset="PIC16F1829" device=""/>
 <part name="XB1" library="maxstream" deviceset="XBEE" device="-PRO"/>
-<part name="GPIO" library="pinhead" deviceset="PINHD-1X8" device="/90"/>
 <part name="C1" library="rcl" deviceset="C-US" device="050-035X075" value="10nF"/>
 <part name="C2" library="rcl" deviceset="C-US" device="050-035X075" value="100nF"/>
@@
 <part name="HEARTBEAT" library="led" deviceset="LED" device="5MM"/>
 <part name="DOOR_OPEN" library="led" deviceset="LED" device="5MM"/>
-<part name="R2" library="rcl" deviceset="R-US_" device="0309/12" value="1K"/>
+<part name="R2" library="rcl" deviceset="R-US_" device="0309/12" value="10K"/>
 <part name="R3" library="rcl" deviceset="R-US_" device="0309/12" value="1K"/>
 <part name="U$4" library="fritz" deviceset="BUZZER" device=""/>
 <part name="X1" library="con-wago-508" deviceset="W237-02P" device=""/>
 <part name="R4" library="rcl" deviceset="R-US_" device="0309/12" value="10K"/>
+<part name="JP1" library="pinhead" deviceset="PINHD-1X10" device=""/>
+<part name="U$5" library="fritz" deviceset="SWITCH_MOMENTARY" device=""/>
+<part name="R5" library="rcl" deviceset="R-US_" device="0309/12" value="10K"/>
 </parts>
 <sheets>
@@
 <instance part="U$1" gate="G$1" x="27.94" y="99.06"/>
 <instance part="XB1" gate="G$1" x="142.24" y="104.14"/>
-<instance part="GPIO" gate="A" x="12.7" y="55.88"/>
 <instance part="C1" gate="G$1" x="38.1" y="66.04"/>
 <instance part="C2" gate="G$1" x="50.8" y="66.04"/>
@@
 <instance part="R2" gate="G$1" x="116.84" y="63.5" rot="R180"/>
 <instance part="R3" gate="G$1" x="116.84" y="50.8" rot="R180"/>
-<instance part="U$4" gate="G$1" x="106.68" y="35.56"/>
+<instance part="U$4" gate="G$1" x="106.68" y="35.56" rot="MR0"/>
 <instance part="X1" gate="-1" x="-22.86" y="25.4"/>
 <instance part="X1" gate="-2" x="-22.86" y="20.32"/>
 <instance part="R4" gate="G$1" x="-15.24" y="33.02" rot="R90"/>
+<instance part="JP1" gate="A" x="12.7" y="60.96"/>
+<instance part="U$5" gate="G$1" x="68.58" y="17.78"/>
+<instance part="R5" gate="G$1" x="58.42" y="25.4" rot="R90"/>
 </instances>
 <busses>
@@
 <wire x1="-15.24" y1="38.1" x2="-15.24" y2="40.64" width="0.1524" layer="91"/>
 <label x="-17.78" y="40.64" size="1.778" layer="95"/>
+</segment>
+<segment>
+<pinref part="JP1" gate="A" pin="2"/>
+<wire x1="10.16" y1="68.58" x2="2.54" y2="68.58" width="0.1524" layer="91"/>
+<label x="-2.54" y="68.58" size="1.778" layer="95"/>
+</segment>
+<segment>
+<pinref part="U$4" gate="G$1" pin="2"/>
+<wire x1="101.6" y1="33.02" x2="119.38" y2="33.02" width="0.1524" layer="91"/>
+<label x="119.38" y="33.02" size="1.778" layer="95"/>
+</segment>
+<segment>
+<pinref part="R5" gate="G$1" pin="2"/>
+<wire x1="58.42" y1="30.48" x2="58.42" y2="33.02" width="0.1524" layer="91"/>
+<label x="55.88" y="33.02" size="1.778" layer="95"/>
 </segment>
 </net>
@@
 </segment>
 <segment>
-<pinref part="U$4" gate="G$1" pin="2"/>
-<wire x1="111.76" y1="33.02" x2="119.38" y2="33.02" width="0.1524" layer="91"/>
-<label x="119.38" y="33.02" size="1.778" layer="95"/>
-</segment>
-<segment>
 <pinref part="X1" gate="-2" pin="KL"/>
 <wire x1="-17.78" y1="20.32" x2="-12.7" y2="20.32" width="0.1524" layer="91"/>
 <label x="-12.7" y="20.32" size="1.778" layer="95"/>
 </segment>
+<segment>
+<pinref part="JP1" gate="A" pin="1"/>
+<wire x1="10.16" y1="71.12" x2="2.54" y2="71.12" width="0.1524" layer="91"/>
+<label x="-2.54" y="71.12" size="1.778" layer="95"/>
+</segment>
+<segment>
+<pinref part="U$5" gate="G$1" pin="2"/>
+<wire x1="73.66" y1="17.78" x2="78.74" y2="17.78" width="0.1524" layer="91"/>
+<label x="78.74" y="17.78" size="1.778" layer="95"/>
+</segment>
 </net>
 <net name="RX" class="0">
@@
 <segment>
 <pinref part="U$4" gate="G$1" pin="1"/>
-<wire x1="101.6" y1="33.02" x2="93.98" y2="33.02" width="0.1524" layer="91"/>
+<wire x1="111.76" y1="33.02" x2="93.98" y2="33.02" width="0.1524" layer="91"/>
 <label x="83.82" y="33.02" size="1.778" layer="95"/>
 </segment>
@@
 </segment>
 <segment>
-<pinref part="GPIO" gate="A" pin="1"/>
-<wire x1="10.16" y1="66.04" x2="0" y2="66.04" width="0.1524" layer="91"/>
-<label x="-10.16" y="66.04" size="1.778" layer="95"/>
-</segment>
-<segment>
 <pinref part="HEARTBEAT" gate="G$1" pin="A"/>
 <wire x1="101.6" y1="63.5" x2="93.98" y2="63.5" width="0.1524" layer="91"/>
 <label x="83.82" y="63.5" size="1.778" layer="95"/>
 </segment>
+<segment>
+<pinref part="JP1" gate="A" pin="3"/>
+<wire x1="10.16" y1="66.04" x2="2.54" y2="66.04" width="0.1524" layer="91"/>
+<label x="-5.08" y="66.04" size="1.778" layer="95"/>
+</segment>
 </net>
 <net name="GPIO_1" class="0">
@@
 </segment>
 <segment>
-<pinref part="GPIO" gate="A" pin="2"/>
-<wire x1="10.16" y1="63.5" x2="0" y2="63.5" width="0.1524" layer="91"/>
-<label x="-10.16" y="63.5" size="1.778" layer="95"/>
-</segment>
-<segment>
 <pinref part="DOOR_OPEN" gate="G$1" pin="A"/>
 <wire x1="101.6" y1="50.8" x2="93.98" y2="50.8" width="0.1524" layer="91"/>
 <label x="83.82" y="50.8" size="1.778" layer="95"/>
 </segment>
+<segment>
+<pinref part="JP1" gate="A" pin="4"/>
+<wire x1="10.16" y1="63.5" x2="2.54" y2="63.5" width="0.1524" layer="91"/>
+<label x="-5.08" y="63.5" size="1.778" layer="95"/>
+</segment>
 </net>
 <net name="GPIO_2" class="0">
@@
 </segment>
 <segment>
-<pinref part="GPIO" gate="A" pin="3"/>
-<wire x1="10.16" y1="60.96" x2="0" y2="60.96" width="0.1524" layer="91"/>
-<label x="-10.16" y="60.96" size="1.778" layer="95"/>
+<pinref part="JP1" gate="A" pin="5"/>
+<wire x1="10.16" y1="60.96" x2="2.54" y2="60.96" width="0.1524" layer="91"/>
+<label x="-5.08" y="60.96" size="1.778" layer="95"/>
+</segment>
+<segment>
+<pinref part="U$5" gate="G$1" pin="1"/>
+<wire x1="63.5" y1="17.78" x2="58.42" y2="17.78" width="0.1524" layer="91"/>
+<wire x1="58.42" y1="17.78" x2="58.42" y2="20.32" width="0.1524" layer="91"/>
+<wire x1="58.42" y1="17.78" x2="55.88" y2="17.78" width="0.1524" layer="91"/>
+<pinref part="R5" gate="G$1" pin="1"/>
+<label x="48.26" y="17.78" size="1.778" layer="95"/>
 </segment>
 </net>
@@
 </segment>
 <segment>
-<pinref part="GPIO" gate="A" pin="8"/>
-<wire x1="10.16" y1="48.26" x2="0" y2="48.26" width="0.1524" layer="91"/>
-<label x="-10.16" y="48.26" size="1.778" layer="95"/>
+<pinref part="JP1" gate="A" pin="10"/>
+<wire x1="10.16" y1="48.26" x2="2.54" y2="48.26" width="0.1524" layer="91"/>
+<label x="-5.08" y="48.26" size="1.778" layer="95"/>
 </segment>
 </net>
@@
 </segment>
 <segment>
-<pinref part="GPIO" gate="A" pin="7"/>
-<wire x1="10.16" y1="50.8" x2="0" y2="50.8" width="0.1524" layer="91"/>
-<label x="-10.16" y="50.8" size="1.778" layer="95"/>
+<pinref part="JP1" gate="A" pin="9"/>
+<wire x1="10.16" y1="50.8" x2="2.54" y2="50.8" width="0.1524" layer="91"/>
+<label x="-5.08" y="50.8" size="1.778" layer="95"/>
 </segment>
 </net>
@@
 </segment>
 <segment>
-<pinref part="GPIO" gate="A" pin="4"/>
-<wire x1="10.16" y1="58.42" x2="0" y2="58.42" width="0.1524" layer="91"/>
-<label x="-10.16" y="58.42" size="1.778" layer="95"/>
+<pinref part="JP1" gate="A" pin="6"/>
+<wire x1="10.16" y1="58.42" x2="2.54" y2="58.42" width="0.1524" layer="91"/>
+<label x="-5.08" y="58.42" size="1.778" layer="95"/>
 </segment>
 </net>
@@
 </segment>
 <segment>
-<pinref part="GPIO" gate="A" pin="5"/>
-<wire x1="10.16" y1="55.88" x2="0" y2="55.88" width="0.1524" layer="91"/>
-<label x="-10.16" y="55.88" size="1.778" layer="95"/>
+<pinref part="JP1" gate="A" pin="7"/>
+<wire x1="10.16" y1="55.88" x2="2.54" y2="55.88" width="0.1524" layer="91"/>
+<label x="-5.08" y="55.88" size="1.778" layer="95"/>
 </segment>
 </net>
@@
 </segment>
 <segment>
-<pinref part="GPIO" gate="A" pin="6"/>
-<wire x1="10.16" y1="53.34" x2="0" y2="53.34" width="0.1524" layer="91"/>
-<label x="-10.16" y="53.34" size="1.778" layer="95"/>
+<pinref part="JP1" gate="A" pin="8"/>
+<wire x1="10.16" y1="53.34" x2="2.54" y2="53.34" width="0.1524" layer="91"/>
+<label x="-5.08" y="53.34" size="1.778" layer="95"/>
 </segment>
 </net>
@@
 <label x="-40.64" y="53.34" size="1.778" layer="95"/>
 </segment>
+<segment>
+<pinref part="U$1" gate="G$1" pin="RA0/ICSPDAT"/>
+<wire x1="53.34" y1="109.22" x2="58.42" y2="109.22" width="0.1524" layer="91"/>
+<label x="58.42" y="109.22" size="1.778" layer="95"/>
+</segment>
 </net>
 <net name="ICSPCLK" class="0">
@@
 <label x="-40.64" y="50.8" size="1.778" layer="95"/>
 </segment>
-</net>
+<segment>
+<pinref part="U$1" gate="G$1" pin="RA1/ICSPCLK"/>
+<wire x1="53.34" y1="106.68" x2="58.42" y2="106.68" width="0.1524" layer="91"/>
+<label x="58.42" y="106.68" size="1.778" layer="95"/>
+</segment>
+</net>

Commit message: max_bell done
Connections:
- new net BUTTON: R5.1, U$1.RA2, U$5.1
- net GPIO_2: no longer R5.1, U$5.1
Changed lines of the file:
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@@
 <label x="-5.08" y="60.96" size="1.778" layer="95"/>
-</segment>
-<segment>
-<pinref part="U$5" gate="G$1" pin="1"/>
-<wire x1="63.5" y1="17.78" x2="58.42" y2="17.78" width="0.1524" layer="91"/>
-<wire x1="58.42" y1="17.78" x2="58.42" y2="20.32" width="0.1524" layer="91"/>
-<wire x1="58.42" y1="17.78" x2="55.88" y2="17.78" width="0.1524" layer="91"/>
-<pinref part="R5" gate="G$1" pin="1"/>
-<label x="48.26" y="17.78" size="1.778" layer="95"/>
 </segment>
 </net>
@@
 </segment>
 </net>
+<net name="BUTTON" class="0">
+<segment>
+<pinref part="U$1" gate="G$1" pin="RA2"/>
+<wire x1="53.34" y1="104.14" x2="58.42" y2="104.14" width="0.1524" layer="91"/>
+<label x="58.42" y="104.14" size="1.778" layer="95"/>
+</segment>
+<segment>
+<pinref part="U$5" gate="G$1" pin="1"/>
+<wire x1="63.5" y1="17.78" x2="58.42" y2="17.78" width="0.1524" layer="91"/>
+<wire x1="58.42" y1="17.78" x2="58.42" y2="20.32" width="0.1524" layer="91"/>
+<wire x1="58.42" y1="17.78" x2="55.88" y2="17.78" width="0.1524" layer="91"/>
+<pinref part="R5" gate="G$1" pin="1"/>
+<label x="45.72" y="17.78" size="1.778" layer="95"/>
+</segment>
+</net>
